Commit message: clean all, write setup.py, License, use qibullet class Signed-off-by: mcaniot <maxime.caniot@gmail.com>

File: modular_sphere/data/robot_sphere.urdf (robot description, URDF)
Before this commit: robot urdf_robot, 1 links, 0 joints
Links:
- link baseLink: geometry collision sphere radius=0.5; visual mesh filename=robot_sphere.obj scale=0.5 0.5 0.5

Commit message: update size and mass

File: modular_sphere/data/robot_sphere.urdf (robot description, URDF)
Before this commit: robot robot_sphere, 1 links, 0 joints
Links:
- link baseLink: mass 10.0 -> 0.300; geometry collision sphere radius=0.10; visual mesh filename=robot_sphere.obj scale=0.10 0.10 0.10
